File: COFFEE_MAKER/ESP32-Breakout.kicad_sch (KiCad schematic)
At the start: 0 parts

Commit message: update accuracy
Parts:
- added C1 (x2): 1uF, Capacitor_SMD:C_0805_2012Metric_Pad1.18x1.45mm_HandSolder, symbol Device:C
- added C11: 10uF, Capacitor_SMD:C_1206_3216Metric_Pad1.33x1.80mm_HandSolder, symbol Device:C
- added C12: 22uF, Capacitor_SMD:C_0805_2012Metric_Pad1.18x1.45mm_HandSolder, symbol Device:C
- added D1: PESD12VL2BT, Package_TO_SOT_SMD:SOT-23, symbol Power_Protection:SP0502BAHT
- added D2: D_Schottky, Diode_SMD:D_SOD-128, symbol Device:D_Schottky
- added D3: GREEN, LED_SMD:LED_1206_3216Metric_Pad1.42x1.75mm_HandSolder, symbol Device:LED
- added J3: USB_B_Micro, Connector_USB:USB_Micro-B_Amphenol_10103594-0001LF_Horizontal, symbol Connector:USB_B_Micro
- added R21: 10k, Resistor_SMD:R_0805_2012Metric_Pad1.20x1.40mm_HandSolder, symbol Device:R
- added R22: 300, Resistor_SMD:R_0805_2012Metric_Pad1.20x1.40mm_HandSolder, symbol Device:R
- added SW1, SW2: 1825910-6, 1825910-6:SW_1825910-6-4, symbol 1825910-6:1825910-6
- added U10: ESP32-S3-WROOM-1-N16R2, RF_Module:ESP32-S3-WROOM-1, symbol ESP32-S3-WROOM-1-N16R2:ESP32-S3-WROOM-1-N16R2
- added U9: AZ1084-3.3, Package_TO_SOT_SMD:TO-252-2, symbol Regulator_Linear:AZ1084-3.3
Connections:
- new net: D2.2 (A), J3.1 (VBUS)
- new net: D3.2 (A), R22.1
- new net +3.3V: C12.1, R21.1, R22.2, U10.2 (3V3), U9.2 (VO)
- new net +5V: C11.1, D2.1 (K), U9.3 (VI)
- new net BOOT: C1.2, SW1.3, SW1.4, U10.27 (IO0)
- new net EN: C1.2, R21.2, SW2.3, SW2.4, U10.3 (EN)
- new net GND: C1.1, C1.1, C11.2, C12.2, D1.3 (A), D3.1 (K), J3.5 (GND), J3.6 (Shield), SW1.1, SW1.2, SW2.1, SW2.2, U10.1 (GND), U10.40 (GND__1), U10.41 (GND__2), U9.1 (GND)
- new net IO1: U10.39 (IO1)
- new net IO10: U10.18 (IO10)
- new net IO11: U10.19 (IO11)
- new net IO12: U10.20 (IO12)
- new net IO13: U10.21 (IO13)
- new net IO14: U10.22 (IO14)
- new net IO15: U10.8 (IO15)
- new net IO16: U10.9 (IO16)
- new net IO17: U10.10 (IO17)
- new net IO18: U10.11 (IO18)
- new net IO2: U10.38 (IO2)
- new net IO21: U10.23 (IO21)
- new net IO38: U10.31 (IO38)
- new net IO39: U10.32 (IO39)
- new net IO4: U10.4 (IO4)
- new net IO40: U10.33 (IO40)
- new net IO41: U10.34 (IO41)
- new net IO42: U10.35 (IO42)
- new net IO47: U10.24 (IO47)
- new net IO48: U10.25 (IO48)
- new net IO5: U10.5 (IO5)
- new net IO6: U10.6 (IO6)
- new net IO7: U10.7 (IO7)
- new net IO8: U10.12 (IO8)
- new net IO9: U10.17 (IO9)
- new net USB_D+: D1.1 (K), J3.3 (D+), U10.14 (IO20)
- new net USB_D-: D1.2 (K), J3.2 (D-), U10.13 (IO19)
- no-connect marks 0 -> 9
Other:
- note added: "Micro-USB"
