File: COFFEE_MAKER/COFFEE_MAKER.kicad_sch (KiCad schematic)
At the start: 54 parts, among them J1 Conn_01x03_Pin, J2 Conn_01x06, J3 Conn_01x03_Pin, J4 Screw_Terminal_01x02, J5 USB_C_Receptacle_USB2.0_16P, J7 Conn_01x04, Q1 BC850, SW5 Reset, SW6 Boot, U3 AMS1117-3.3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

Commit message: schematic footprints assigned
Parts:
- removed C9: C, symbol Device:C
- added C5: 0.01 uF, Capacitor_SMD:C_0805_2012Metric, symbol Device:C
- C10: value C -> 0.1uF; footprint (none) -> Capacitor_SMD:C_0805_2012Metric
- C13, C14: value C_Polarized_US -> 10 uF; footprint (none) -> Capacitor_SMD:C_0805_2012Metric
- C16: value 100nF -> 0.1uF; footprint (none) -> Capacitor_SMD:C_0805_2012Metric
- C17, C18, C19, C20, C21: footprint (none) -> Capacitor_SMD:C_0805_2012Metric
- D1: footprint (none) -> LED_SMD:LED_0805_2012Metric
- FB1, FB2: footprint (none) -> Resistor_SMD:R_0603_1608Metric
- J2: footprint (none) -> Connector_PinHeader_2.00mm:PinHeader_1x06_P2.00mm_Vertical
- J4: footprint (none) -> TerminalBlock_MetzConnect:TerminalBlock_MetzConnect_Type094_RT03502HBLU_1x02_P5.00mm_Horizontal
- J5: footprint (none) -> Connector_USB:USB_C_Receptacle_GCT_USB4125-xx-x-0190_6P_TopMnt_Horizontal
- J7: footprint (none) -> Connector_PinHeader_1.00mm:PinHeader_1x04_P1.00mm_Vertical
- R1: renamed from R3; value R -> 10k; footprint (none) -> Resistor_SMD:R_0603_1608Metric
- R2: renamed from R4; value R -> 10k; footprint (none) -> Resistor_SMD:R_0603_1608Metric
- R3: renamed from R5; value R -> 10k; footprint (none) -> Resistor_SMD:R_0603_1608Metric
- R4: renamed from R6; value R -> 10k; footprint (none) -> Resistor_SMD:R_0603_1608Metric
- R5: renamed from R7; value R -> 10k; footprint (none) -> Resistor_SMD:R_0603_1608Metric
- R6: renamed from R11; value R -> 4.7k; footprint (none) -> Resistor_SMD:R_0805_2012Metric
- R7: renamed from R12; value R -> 4.7k; footprint (none) -> Resistor_SMD:R_0805_2012Metric
- R8: renamed from R13; value R -> 1k; footprint (none) -> Resistor_SMD:R_0805_2012Metric
- R9: renamed from R14; value R -> 4.7k; footprint (none) -> Resistor_SMD:R_0805_2012Metric
- RV1: footprint Potentiometer_SMD:Potentiometer_ACP_CA9-VSMD_Vertical_Hole -> Potentiometer_SMD:Potentiometer_Bourns_TC33X_Vertical
- renumbered R8 to R11, R9 to R12
Connections:
- net at FB2.1, U5.3 (T+): now also C5.1
- net at FB1.2, U5.2 (T-): now also C5.2
Other:
- note added: "Voltage Drop down Regulators"
- moved on the sheet: R1

Commit message: schematics done (custom footprint PCF8574 and ESP32-S2-N4)
Parts:
- JP1, JP2, JP3: footprint (none) -> Jumper:SolderJumper-3_P1.3mm_Open_Pad1.0x1.5mm
- JP4: footprint (none) -> Jumper:SolderJumper-3_P1.3mm_Open_RoundedPad1.0x1.5mm
- R10: footprint (none) -> Resistor_SMD:R_0603_1608Metric
- R11, R12: footprint (none) -> Resistor_SMD:R_0805_2012Metric
- SW5, SW6: footprint (none) -> Button_Switch_SMD:SW_SPST_TL3305A
- U4: footprint (none) -> PCF8574:SOIC16R
- U8: footprint PCM_Espressif:ESP32-S2-SOLO -> ESP32-S2-SOLO-U-N4R2:XCVR_ESP32-S2-SOLO-U-N4R2
Changed lines of the file:
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@@
       (effects (font (size 1.27 1.27)))
     )
-    (property "Footprint" "" (at -199.39 27.178 90)
-      (effects (font (size 1.27 1.27)) hide)
-    )
-    (property "Datasheet" "~" (at -199.39 25.4 0)
+    (property "Footprint" "Resistor_SMD:R_0805_2012Metric" (at -199.39 27.178 90)
+      (effects (font (size 1.27 1.27)) hide)
+    )
+    (property "Datasheet" "https://www.yageo.com/upload/media/product/products/datasheet/rchip/PYu-RC_Group_51_RoHS_L_12.pdf" (at -199.39 25.4 0)
       (effects (font (size 1.27 1.27)) hide)
     )
@@
   )
   (symbol (lib_id "Jumper:SolderJumper_2_Open") (at 34.29 34.29 0) (unit 1)
-    (in_bom yes) (on_board yes) (dnp no) (fields_autoplaced)
-    (property "Reference" "JP1" (at 34.29 27.94 0)
-      (effects (font (size 1.27 1.27)))
-    )
-    (property "Value" "A0" (at 34.29 30.48 0)
-      (effects (font (size 1.27 1.27)))
-    )
-    (property "Footprint" "" (at 34.29 34.29 0)
+    (in_bom yes) (on_board yes) (dnp no)
+    (property "Reference" "JP1" (at 34.29 35.56 0)
+      (effects (font (size 1.27 1.27)))
+    )
+    (property "Value" "A0" (at 34.29 36.83 0)
+      (effects (font (size 1.27 1.27)))
+    )
+    (property "Footprint" "Jumper:SolderJumper-3_P1.3mm_Open_Pad1.0x1.5mm" (at 34.29 34.29 0)
       (effects (font (size 1.27 1.27)) hide)
     )
@@
       (effects (font (size 1.27 1.27)) (justify left))
     )
-    (property "Footprint" "" (at 119.38 49.53 0)
+    (property "Footprint" "PCF8574:SOIC16R" (at 119.38 49.53 0)
       (effects (font (size 1.27 1.27)) hide)
     )
@@
       (effects (font (size 1.27 1.27)) (justify right))
     )
-    (property "Footprint" "" (at 99.06 67.31 0)
+    (property "Footprint" "Jumper:SolderJumper-3_P1.3mm_Open_RoundedPad1.0x1.5mm" (at 99.06 67.31 0)
       (effects (font (size 1.27 1.27)) hide)
     )
@@
   (symbol (lib_id "Jumper:SolderJumper_2_Open") (at 34.29 40.64 0) (unit 1)
     (in_bom yes) (on_board yes) (dnp no)
-    (property "Reference" "JP2" (at 34.29 34.29 0)
-      (effects (font (size 1.27 1.27)))
-    )
-    (property "Value" "A1" (at 34.29 36.83 0)
-      (effects (font (size 1.27 1.27)))
-    )
-    (property "Footprint" "" (at 34.29 40.64 0)
+    (property "Reference" "JP2" (at 34.29 41.91 0)
+      (effects (font (size 1.27 1.27)))
+    )
+    (property "Value" "A1" (at 34.29 43.18 0)
+      (effects (font (size 1.27 1.27)))
+    )
+    (property "Footprint" "Jumper:SolderJumper-3_P1.3mm_Open_Pad1.0x1.5mm" (at 34.29 40.64 0)
       (effects (font (size 1.27 1.27)) hide)
     )
@@
       (effects (font (size 1.27 1.27)) (justify left))
     )
-    (property "Footprint" "PCM_Espressif:ESP32-S2-SOLO" (at -104.14 127 0)
+    (property "Footprint" "ESP32-S2-SOLO-U-N4R2:XCVR_ESP32-S2-SOLO-U-N4R2" (at -104.14 127 0)
       (effects (font (size 1.27 1.27)) hide)
     )
@@
       (effects (font (size 1.27 1.27)) (justify left))
     )
-    (property "Footprint" "" (at -163.068 29.21 90)
+    (property "Footprint" "Resistor_SMD:R_0603_1608Metric" (at -163.068 29.21 90)
       (effects (font (size 1.27 1.27)) hide)
     )
@@
       (effects (font (size 1.27 1.27)))
     )
-    (property "Footprint" "" (at -170.18 30.48 0)
+    (property "Footprint" "Button_Switch_SMD:SW_SPST_TL3305A" (at -170.18 30.48 0)
       (effects (font (size 1.27 1.27)) hide)
     )
@@
       (effects (font (size 1.27 1.27)))
     )
-    (property "Footprint" "" (at -199.39 32.512 90)
+    (property "Footprint" "Resistor_SMD:R_0805_2012Metric" (at -199.39 32.512 90)
       (effects (font (size 1.27 1.27)) hide)
     )
@@
   )
   (symbol (lib_id "Jumper:SolderJumper_2_Open") (at 34.29 46.99 0) (unit 1)
-    (in_bom yes) (on_board yes) (dnp no) (fields_autoplaced)
-    (property "Reference" "JP3" (at 34.29 40.64 0)
-      (effects (font (size 1.27 1.27)))
-    )
-    (property "Value" "A2" (at 34.29 43.18 0)
-      (effects (font (size 1.27 1.27)))
-    )
-    (property "Footprint" "" (at 34.29 46.99 0)
+    (in_bom yes) (on_board yes) (dnp no)
+    (property "Reference" "JP3" (at 34.29 49.53 0)
+      (effects (font (size 1.27 1.27)))
+    )
+    (property "Value" "A2" (at 34.29 50.8 0)
+      (effects (font (size 1.27 1.27)))
+    )
+    (property "Footprint" "Jumper:SolderJumper-3_P1.3mm_Open_Pad1.0x1.5mm" (at 34.29 46.99 0)
       (effects (font (size 1.27 1.27)) hide)
     )
@@
       (effects (font (size 1.27 1.27)))
     )
-    (property "Footprint" "" (at -34.29 45.72 0)
-      (effects (font (size 1.27 1.27)) hide)
-    )
+    (property "Footprint" "Button_Switch_SMD:SW_SPST_TL3305A" (at -34.29 45.72 0)
+      (effects (font (size 1.27 1.27)) hide)
+    )

Commit message: update esp32 footprint, layout wip
Parts:
- removed U3: AMS1117-3.3, Package_TO_SOT_SMD:SOT-223-3_TabPin2, symbol Regulator_Linear:AMS1117-3.3
- removed U6: AMS1117-5.0, Package_TO_SOT_SMD:SOT-223-3_TabPin2, symbol Regulator_Linear:AMS1117-5.0
- added U1: OKI-78SR-3.3_1.5-W36H-C, Converter_DCDC:Converter_DCDC_Murata_OKI-78SR_Horizontal, symbol Converter_DCDC:OKI-78SR-3.3_1.5-W36H-C
- added U2: OKI-78SR-5_1.5-W36-C, Converter_DCDC:Converter_DCDC_Murata_OKI-78SR_Horizontal, symbol Converter_DCDC:OKI-78SR-5_1.5-W36-C
- J5: footprint Connector_USB:USB_C_Receptacle_GCT_USB4125-xx-x-0190_6P_TopMnt_Horizontal -> Connector_USB:USB_C_Receptacle_GCT_USB4105-xx-A_16P_TopMnt_Horizontal
- JP1, JP2, JP3: footprint Jumper:SolderJumper-3_P1.3mm_Open_Pad1.0x1.5mm -> Jumper:SolderJumper-2_P1.3mm_Open_RoundedPad1.0x1.5mm
- JP4: footprint Jumper:SolderJumper-3_P1.3mm_Open_RoundedPad1.0x1.5mm -> Jumper:SolderJumper-2_P1.3mm_Open_RoundedPad1.0x1.5mm
- U8: footprint ESP32-S2-SOLO-U-N4R2:XCVR_ESP32-S2-SOLO-U-N4R2 -> ESP32-S2-SOLO-U-N4R2:ESP32-S2-SOLO
Connections:
- net GND: now also U1.2 (GND), U2.2 (GND)
- net V_ALL+: now also U1.1 (IN), U2.1 (IN)
- net at F1.1: now also U1.3 (OUT)
- net at F2.1: now also U2.3 (OUT)

Commit message: board layout wip 27 errors
Connections:
- net +3.3V is gone; now on net +3V3: C17.1, C19.2, C20.2, C3.2, F1.2, J1.1 (Pin_1), J3.1 (Pin_1), R10.1, U7.2 (VO), U8.2 (3V3)

Commit message: layout done, saved copy of slides
.Layout done, slides saved as ppt and pdf in folder, google slides here:
https://docs.google.com/presentation/d/1jqAALReZK5NcbOIQpBx0YGVnQ22f8MZOJf6NqvKvuig/edit#slide=id.g26e1c898e73_0_26
Parts:
- J7: footprint Connector_PinHeader_1.00mm:PinHeader_1x04_P1.00mm_Vertical -> Connector_PinHeader_2.00mm:PinHeader_1x04_P2.00mm_Vertical
Changed lines of the file:
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@@
     )
     (property "Footprint" "ESP32-S2-SOLO-U-N4R2:ESP32-S2-SOLO" (at -104.14 127 0)
-      (effects (font (size 1.27 1.27)) hide)
+      (effects (font (size 1.27 1.27)))
     )
     (property "Datasheet" "https://www.espressif.com/sites/default/files/documentation/esp32-s2-solo_esp32-s2-solo-u_datasheet_en.pdf" (at -104.14 129.54 0)
@@
       (effects (font (size 1.27 1.27)))
     )
-    (property "Footprint" "Connector_PinHeader_1.00mm:PinHeader_1x04_P1.00mm_Vertical" (at 20.32 105.41 0)
-      (effects (font (size 1.27 1.27)) hide)
-    )
+    (property "Footprint" "Connector_PinHeader_2.00mm:PinHeader_1x04_P2.00mm_Vertical" (at 20.32 105.41 0)
+      (effects (font (size 1.27 1.27)) hide)
+    )

Commit message: schematic bom wip
Parts:
- C1, C2: footprint Capacitor_SMD:C_0603_1608Metric -> Capacitor_SMD:C_0805_2012Metric
- C13, C14: value 10 uF -> 10uF
- C18, C20, C21: value .1uF -> 0.1uF
- C5: value 0.01 uF -> 0.01uF
- R11, R12: value 5.1 k -> 5.1k
Changed lines of the file:
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@@
       (effects (font (size 1.27 1.27)) hide)
     )
-    (property "Datasheet" "~" (at 254 60.96 0)
+    (property "Datasheet" "https://search.murata.co.jp/Ceramy/image/img/A01X/G101/ENG/GRM188R60J226MEA0-01.pdf" (at 254 60.96 0)
       (effects (font (size 1.27 1.27)) hide)
     )
@@
       (effects (font (size 1.27 1.27)))
     )
-    (property "Value" "5.1 k" (at -199.39 21.59 90)
+    (property "Value" "5.1k" (at -199.39 21.59 90)
       (effects (font (size 1.27 1.27)))
     )
@@
       (effects (font (size 1.27 1.27)) (justify left) hide)
     )
-    (property "Datasheet" "~" (at 236.22 22.86 0)
+    (property "Datasheet" "https://www.belfuse.com/resources/datasheets/circuitprotection/ds-cp-c2q-series.pdf" (at 236.22 22.86 0)
       (effects (font (size 1.27 1.27)) hide)
     )
@@
       (effects (font (size 1.27 1.27)) (justify left))
     )
-    (property "Value" "10 uF" (at 201.93 154.305 0)
+    (property "Value" "10uF" (at 201.93 154.305 0)
       (effects (font (size 1.27 1.27)) (justify left))
     )
@@
       (effects (font (size 1.27 1.27)) (justify left) hide)
     )
-    (property "Datasheet" "~" (at 251.46 55.88 0)
+    (property "Datasheet" "https://www.belfuse.com/resources/datasheets/circuitprotection/ds-cp-c2q-series.pdf" (at 251.46 55.88 0)
       (effects (font (size 1.27 1.27)) hide)
     )
@@
       (effects (font (size 1.27 1.27)) (justify left))
     )
-    (property "Value" "0.01 uF" (at 210.82 130.81 0)
+    (property "Value" "0.01uF" (at 210.82 130.81 0)
       (effects (font (size 1.27 1.27)) (justify left))
     )
@@
       (effects (font (size 1.27 1.27)) hide)
     )
-    (property "Datasheet" "~" (at -104.14 21.59 0)
+    (property "Datasheet" "https://mm.digikey.com/Volume0/opasdata/d220001/medias/docus/1105/CL21B105KAFNNNE_Spec.pdf" (at -104.14 21.59 0)
       (effects (font (size 1.27 1.27)) hide)
     )
@@
       (effects (font (size 1.27 1.27)) (justify left))
     )
-    (property "Value" "10 uF" (at 179.07 154.94 0)
+    (property "Value" "10uF" (at 179.07 154.94 0)
       (effects (font (size 1.27 1.27)) (justify left))
     )
@@
       (effects (font (size 1.27 1.27)) (justify right))
     )
-    (property "Footprint" "Capacitor_SMD:C_0603_1608Metric" (at 208.28 30.48 0)
-      (effects (font (size 1.27 1.27)) hide)
-    )
-    (property "Datasheet" "~" (at 208.28 30.48 0)
+    (property "Footprint" "Capacitor_SMD:C_0805_2012Metric" (at 208.28 30.48 0)
+      (effects (font (size 1.27 1.27)) hide)
+    )
+    (property "Datasheet" "https://mm.digikey.com/Volume0/opasdata/d220001/medias/docus/609/CL21A106KOQNNNE_Spec.pdf" (at 208.28 30.48 0)
       (effects (font (size 1.27 1.27)) hide)
     )
@@
       (effects (font (size 1.27 1.27)) hide)
     )
-    (property "Datasheet" "~" (at -229.87 110.49 0)
+    (property "Datasheet" "https://mm.digikey.com/Volume0/opasdata/d220001/medias/docus/893/CL21B104KCFNNNE_Spec.pdf" (at -229.87 110.49 0)
       (effects (font (size 1.27 1.27)) hide)
     )
@@
       (effects (font (size 1.27 1.27)) hide)
     )
-    (property "Datasheet" "~" (at -196.85 110.49 0)
+    (property "Datasheet" "https://mm.digikey.com/Volume0/opasdata/d220001/medias/docus/609/CL21A106KOQNNNE_Spec.pdf" (at -196.85 110.49 0)
       (effects (font (size 1.27 1.27)) hide)
     )
@@
       (effects (font (size 1.27 1.27)) hide)
     )
-    (property "Datasheet" "~" (at 247.65 27.94 0)
+    (property "Datasheet" "https://search.murata.co.jp/Ceramy/image/img/A01X/G101/ENG/GRM188R60J226MEA0-01.pdf" (at 247.65 27.94 0)
       (effects (font (size 1.27 1.27)) hide)
     )
@@
       (effects (font (size 1.27 1.27)) (justify left))
     )
-    (property "Value" ".1uF" (at -87.63 23.495 0)
+    (property "Value" "0.1uF" (at -87.63 23.495 0)
       (effects (font (size 1.27 1.27)) (justify left))
     )
@@
       (effects (font (size 1.27 1.27)) hide)
     )
-    (property "Datasheet" "~" (at -91.44 21.59 0)
+    (property "Datasheet" "https://mm.digikey.com/Volume0/opasdata/d220001/medias/docus/893/CL21B104KCFNNNE_Spec.pdf" (at -91.44 21.59 0)
       (effects (font (size 1.27 1.27)) hide)
     )
@@
       (effects (font (size 1.27 1.27)))
     )
-    (property "Value" "5.1 k" (at -199.39 30.48 90)
+    (property "Value" "5.1k" (at -199.39 30.48 90)
       (effects (font (size 1.27 1.27)))
     )
@@
       (effects (font (size 1.27 1.27)) hide)
     )
-    (property "Datasheet" "~" (at -199.39 34.29 0)
+    (property "Datasheet" "https://www.yageo.com/upload/media/product/products/datasheet/rchip/PYu-RC_Group_51_RoHS_L_12.pdf" (at -199.39 34.29 0)
       (effects (font (size 1.27 1.27)) hide)
     )
@@
       (effects (font (size 1.27 1.27)))
     )
-    (property "Value" ".1uF" (at -34.29 57.15 90)
+    (property "Value" "0.1uF" (at -34.29 57.15 90)
       (effects (font (size 1.27 1.27)))
     )
@@
       (effects (font (size 1.27 1.27)) hide)
     )
-    (property "Datasheet" "~" (at -34.29 60.96 0)
+    (property "Datasheet" "https://mm.digikey.com/Volume0/opasdata/d220001/medias/docus/893/CL21B104KCFNNNE_Spec.pdf" (at -34.29 60.96 0)
       (effects (font (size 1.27 1.27)) hide)
     )
@@
       (effects (font (size 1.27 1.27)) (justify right))
     )
-    (property "Footprint" "Capacitor_SMD:C_0603_1608Metric" (at 210.82 63.5 0)
-      (effects (font (size 1.27 1.27)) hide)
-    )
-    (property "Datasheet" "~" (at 210.82 63.5 0)
+    (property "Footprint" "Capacitor_SMD:C_0805_2012Metric" (at 210.82 63.5 0)
+      (effects (font (size 1.27 1.27)) hide)
+    )
+    (property "Datasheet" "https://mm.digikey.com/Volume0/opasdata/d220001/medias/docus/609/CL21A106KOQNNNE_Spec.pdf" (at 210.82 63.5 0)
       (effects (font (size 1.27 1.27)) hide)
     )
@@
       (effects (font (size 1.27 1.27)) hide)
     )
-    (property "Datasheet" "~" (at 31.75 21.59 0)
+    (property "Datasheet" "https://www.we-online.com/components/products/datasheet/150080RS75000.pdf" (at 31.75 21.59 0)
       (effects (font (size 1.27 1.27)) hide)
     )
@@
       (effects (font (size 1.27 1.27)))
     )
-    (property "Value" ".1uF" (at -170.18 40.64 90)
+    (property "Value" "0.1uF" (at -170.18 40.64 90)
       (effects (font (size 1.27 1.27)))
     )
@@
       (effects (font (size 1.27 1.27)) hide)
     )
-    (property "Datasheet" "~" (at -170.18 44.45 0)
-      (effects (font (size 1.27 1.27)) hide)
-    )
+    (property "Datasheet" "https://mm.digikey.com/Volume0/opasdata/d220001/medias/docus/893/CL21B104KCFNNNE_Spec.pdf" (at -170.18 44.45 0)
+      (effects (font (size 1.27 1.27)) hide)
+    )

Commit message: layout v1 done, slides, BOM, manufacturing folder ready
Parts:
- added J6: Barrel_Jack, Connector_BarrelJack:BarrelJack_CUI_PJ-102AH_Horizontal, symbol Connector:Barrel_Jack
- J2: footprint Connector_PinHeader_2.00mm:PinHeader_1x06_P2.00mm_Vertical -> Connector_PinHeader_2.54mm:PinHeader_1x06_P2.54mm_Vertical
Connections:
- net GND: now also J6.2
- net V_ALL+: now also J6.1
Other:
- note added: "24V Barrel Jack"
- moved on the sheet: J1, J3
